Commit message: Add trifinger_meta, visually-realistic model of meta setup

File: trifinger_simulation/robot_properties_fingers/urdf/edu/trifingernyu_white.urdf (robot description, URDF)
Before this commit: robot trifingeredu, 17 links, 16 joints
Links:
- link finger_lower_link_0: geometry collision mesh filename=package://robot_properties_fingers/meshes/edu/lower_link.stl scale=1 1 1; visual mesh filename=package://robot_properties_fingers/meshes/edu/lower_link.stl scale=1 1 1
- link finger_lower_link_120: geometry collision mesh filename=package://robot_properties_fingers/meshes/edu/lower_link.stl scale=1 1 1; visual mesh filename=package://robot_properties_fingers/meshes/edu/lower_link.stl scale=1 1 1
- link finger_lower_link_240: geometry collision mesh filename=package://robot_properties_fingers/meshes/edu/lower_link.stl scale=1 1 1; visual mesh filename=package://robot_properties_fingers/meshes/edu/lower_link.stl scale=1 1 1
- link finger_tip_link_0: geometry 
- link finger_tip_link_120: geometry 
- link finger_tip_link_240: geometry 
